Commit message: Phase 2 착수: returnbot_sim 패키지 (Gazebo 플러그인 + 브링업)
- gazebo_plugins.xacro: diff_drive / gpu_lidar / imu / joint_state_publisher,
  표준 토픽 /cmd_vel /scan /odom. 마찰은 명세 §8대로 튜닝 시작점.
  description 패키지는 실기 공용 순수 모델로 유지하고 시뮬 태그는 여기에만 둔다.
- gazebo.launch.py: 월드 자동 생성 + 스폰 + ros_gz_bridge + RViz.
- drive_mapping_run.py: /odom 피드백 기반 자동 주행. 손 텔레옵은 매번 다른 맵이
  나와 Phase 3 기준 맵으로 못 쓰므로 재현 가능한 경로로 대체.
- robot_params.xacro: LD19 성능 제원(range/rate) 속성 추가, yaml 동기화 테스트 확장.

아직 미검증 — 다음 커밋에서 실제 기동 결과 반영.

Co-Authored-By: Claude Opus 5 (1M context) <noreply@anthropic.com>

File: returnbot_ws/src/returnbot_description/urdf/robot_params.xacro (robot description, xacro)
@@ -41,4 +41,8 @@
   <xacro:property name="lidar_size_z"      value="0.04"/>
   <xacro:property name="lidar_mass"        value="0.2"/>
+  <!-- LD19 성능 제원 (명세 §3 확정값). Gazebo 센서 플러그인이 이 값을 그대로 쓴다. -->
+  <xacro:property name="lidar_range_max"   value="12.0"/>
+  <xacro:property name="lidar_range_min"   value="0.05"/>
+  <xacro:property name="lidar_scan_rate"   value="10.0"/>
   <xacro:property name="imu_size_x"        value="0.02"/>
   <xacro:property name="imu_size_y"        value="0.02"/>
